Commit message: update description

File: gemini_arm_description/urdf/gemini_arm_description.urdf (robot description, URDF)
Before this commit: robot gemini_arm_description, 7 links, 6 joints
Links:
- link link1: mass 0.429111339765701 -> 0.429111339765699
- link link2: mass 0.302188994279633 -> 0.302188994279634
- link link4: mass 0.305571701729797 -> 0.305571705527713
- link link5: mass 0.109576445134181 -> 0.109581130234744
Joints:
- joint joint2: origin xyz=0 0 0.0599999999999999 rpy=1.57079632679489 4.93038065763132E-29 0 -> xyz=0 0 0.060000000000028 rpy=1.57079632679489 4.93038065763132E-29 0
- joint joint3: origin xyz=0 0.16 0 rpy=0 0 0 -> xyz=0 0.159999999999972 0 rpy=0 0 0
- joint joint4: origin xyz=0 0.0604999999999999 0 rpy=-1.5707963267949 -2.77833251643473E-32 5.14058640557261E-17 -> xyz=0 0.0600000000000281 0 rpy=-1.5707963267949 -9.90895775309162E-32 2.1075722764802E-16
- joint joint5: axis 0 0 -1 -> 0.0247180551163906 0 0.999694462198958; origin xyz=0.0519841120343461 0.00128533886604094 0.205700000000028 rpy=1.5707963267949 4.08640132765619E-15 -1.54607575393743 -> xyz=-0.00127297983849752 0.0514842648033036 0.206200000000001 rpy=1.5707963267949 2.1075722764802E-16 0
- joint joint6: origin xyz=-0.000500000000009104 0.0456999999999731 0.0520000000000012 rpy=-1.5707963267949 1.54607575393742 -5.32136220132745E-14 -> xyz=0.00128533886605591 0.0461999999999435 0.0519841120344026 rpy=-1.5707963267949 -6.70540576712656E-29 -5.88614294757338E-14

Commit message: fix link bug
export URDF

File: gemini_arm_description/urdf/gemini_arm_description.urdf (robot description, URDF)
Before this commit: robot gemini_arm_description, 7 links, 6 joints
Links:
- link link2: mass 0.519627467770511 -> 0.519617444659105
- link link3: mass 0.304597711973766 -> 0.304597711973767
- link link4: mass 0.354329700218231 -> 0.305444920744369
- link link5: mass 0.109559148486022 -> 0.109559148486021
