Commit message: change shorter axis4 link and add shell hiding driver so need to change everything

File: gemini_arm_description/robots/gemini_arm_description.urdf (robot description, URDF)
Before this commit: robot gemini_arm_description, 7 links, 6 joints
Links:
- link base_link: mass 0.538356341355379 -> 0.522120243745957
- link link1: mass 0.429111339765699 -> 0.407686363241537
- link link2: mass 0.302188994279634 -> 0.519627467770511
- link link3: mass 0.304609228794722 -> 0.304597711973766
- link link4: mass 0.305571705527713 -> 0.354329700218231
- link link5: mass 0.109581130234744 -> 0.109559148486022
- link link6: mass 0.0205479341797186 -> 0.0278364815211388
Joints:
- joint joint1: origin xyz=0 0 0.0919999999999988 rpy=0 -5.40931672317945E-57 0 -> xyz=0 0 0.101999999999998 rpy=0 0 0
- joint joint2: axis 0.0247180551164637 0 0.999694462198956 -> 0 0 1; origin xyz=0 0 0.060000000000028 rpy=1.57079632679489 4.93038065763132E-29 0 -> xyz=0 0 0.0499999999999997 rpy=1.57079632679489 0 0
- joint joint3: axis 0.0247180551164622 0 0.999694462198956 -> 0 0 1; origin xyz=0 0.159999999999972 0 rpy=0 0 0 -> xyz=0 0.16 0 rpy=0 0 0
- joint joint4: axis 0 0 1 -> 0 0 -1; origin xyz=0 0.0600000000000281 0 rpy=-1.5707963267949 -9.90895775309162E-32 2.1075722764802E-16 -> xyz=0.0468673533334532 -0.063489360827598 -0.0297539470834349 rpy=-1.5707963267949 0 -3.14159265358979
- joint joint5: axis 0.0247180551163906 0 0.999694462198958 -> 0 0 -1; origin xyz=-0.00127297983849752 0.0514842648033036 0.206200000000001 rpy=1.5707963267949 2.1075722764802E-16 0 -> xyz=0.0468673533334465 -0.0817539470834755 -0.289689360827598 rpy=1.5707963267949 -1.83186799063149E-15 -3.14159265358979
- joint joint6: origin xyz=0.00128533886605591 0.0461999999999435 0.0519841120344026 rpy=-1.5707963267949 -6.70540576712656E-29 -5.88614294757338E-14 -> xyz=0 -0.0457 0.052 rpy=1.5707963267949 -3.18770542568412E-16 -2.2904450444239E-15

Commit message: yeah

File: gemini_arm_description/robots/gemini_arm_description.urdf (robot description, URDF)
Before this commit: robot gemini_arm_description, 7 links, 6 joints
Links:
- link link2: mass 0.519617444659105 -> 0.519627467770511
- link link4: mass 0.305444920744369 -> 0.305449608651427
Joints:
- joint joint4: axis 0 0 -1 -> 0 0 1; origin xyz=0.0468673533334532 -0.063489360827598 -0.0297539470834349 rpy=-1.5707963267949 0 -3.14159265358979 -> xyz=0 0.06 0 rpy=-1.5707963267949 0 0
- joint joint5: axis 0 0 -1 -> 0 0 1; origin xyz=0.0468673533334465 -0.0817539470834755 -0.289689360827598 rpy=1.5707963267949 -1.83186799063149E-15 -3.14159265358979 -> xyz=0 0.0520000000000001 0.1662 rpy=1.5707963267949 0 0
- joint joint6: origin xyz=0 -0.0457 0.052 rpy=1.5707963267949 -3.18770542568412E-16 -2.2904450444239E-15 -> xyz=0 0.046199999999943 0.052 rpy=-1.5707963267949 1.55872001956863E-31 1.50753608972822E-15

Commit message: fix time bug and then add some function in python

File: gemini_arm_description/robots/gemini_arm_description.urdf (robot description, URDF)
Before this commit: robot gemini_arm_description, 7 links, 6 joints
Joints:
- joint joint1: limit (none) -> lower=-1.57 upper=1.57 effort=150.0 velocity=4.0
- joint joint2: limit (none) -> lower=-0.8 upper=1.57 effort=150.0 velocity=4.0
- joint joint3: limit (none) -> lower=0 upper=1.57 effort=150.0 velocity=4.0
- joint joint4: limit (none) -> lower=-1.57 upper=1.57 effort=150.0 velocity=4.0
- joint joint5: limit (none) -> lower=0 upper=1.57 effort=150.0 velocity=4.0
- joint joint6: limit (none) -> lower=-3.14 upper=3.14 effort=150.0 velocity=4.0

Commit message: fix joint type to revolute and then joint limit works

File: gemini_arm_description/robots/gemini_arm_description.urdf (robot description, URDF)
Before this commit: robot gemini_arm_description, 7 links, 6 joints
Joints:
- joint joint1: type continuous -> revolute
- joint joint2: type continuous -> revolute
- joint joint3: type continuous -> revolute
- joint joint4: type continuous -> revolute
- joint joint5: type continuous -> revolute
- joint joint6: type continuous -> revolute

Commit message: add pick and place.py

File: gemini_arm_description/robots/gemini_arm_description.urdf (robot description, URDF)
Before this commit: robot gemini_arm_description, 7 links, 6 joints
Joints:
- joint joint5: axis 0 0 1 -> 0 0 -1; limit lower=0 upper=1.57 effort=150.0 velocity=4.0 -> lower=-1.57 upper=1.57 effort=150.0 velocity=4.0
